File: 0035_ADC_Module_ADS1115.kicad_sch (KiCad schematic)
At the start: 11 parts, among them U1 ADS1115IDGS

Commit message: Add files via upload
Parts:
- added D1: LED, LED_SMD:LED_0603_1608Metric, symbol Device:LED
- added J1: Conn_01x04_Socket, Connector_PinSocket_2.54mm:PinSocket_1x04_P2.54mm_Vertical, symbol Connector:Conn_01x04_Socket
- added JP1: Jumper_2_Open, Jumper:SolderJumper-2_P1.3mm_Open_Pad1.0x1.5mm, symbol Jumper:Jumper_2_Open
- added U3: ~, Moduler_:pin_header, symbol moduler_pin:air
- C1, C2, C3: footprint (none) -> Capacitor_SMD:C_0603_1608Metric
- FB1, FB2: footprint (none) -> Inductor_SMD:L_0603_1608Metric
- R1, R3, R4: footprint (none) -> Resistor_SMD:R_0603_1608Metric
- R2: value 0R -> 10k; footprint (none) -> Resistor_SMD:R_0603_1608Metric
- R5: value 10K -> 470r; footprint (none) -> Resistor_SMD:R_0603_1608Metric
- U1: value ADS1115IDGS -> ADS1115
Connections:
- net AIN0: now also J1.4 (Pin_4)
- net AIN1: now also J1.3 (Pin_3)
- net AIN2: now also J1.2 (Pin_2)
- net AIN3: now also J1.1 (Pin_1)
- net GND: now also D1.1 (K), U3.9
- net SCL: now also U3.5
- net SDA: now also U3.6; no longer R1.1, R2.2, U1.1 (ADDR)
- net VCC: no longer C2.1, FB1.1, R2.1, R3.1, R4.1, R5.1
- net at R5.2: now also D1.2 (A); no longer U1.2 (ALERT/RDY)
- new net +5V: C2.1, FB1.1, JP1.2 (B), R2.1, R3.1, R4.1, R5.1, U3.7
- new net ADDR: JP1.1 (A), R1.1, U1.1 (ADDR), U3.12
- new net ALERT: R2.2, U1.2 (ALERT/RDY), U3.13
- no-connect marks 0 -> 12
Other:
- note added: "AIR PIN"
- note added: "I2C PULLUPS"
- note added: "Pin_Out"
- note added: "SENSOR"
- moved on the sheet: C1, C2, C3, FB1, FB2, R1, U1
